Commit message: GCS cok durakli gorev ve gercek donanim ayarlarini entegre et

File: src/marco_description/urdf/properties.xacro (robot description, xacro)
@@ -112,24 +112,18 @@
   <!-- ==================== SENSOR YERLESIMI ==================== -->
   <!--
-    KRITIK / TAHMINI: YDLidar Tmini Pro'nun base_link'e gore konumu.
+    Orange Pi gercek donanim dogrulamasi: YDLidar Tmini Pro'nun base_link'e
+    gore konumu.
     (RPLIDAR A3 DEGIL; eldeki birim Tmini Pro, bkz. AGENT_REFERANS.md)
     laser_link dogru degilse SLAM haritasi ve AMCL lokalizasyonu kayar.
-    CAD'de LiDAR tutucusu YOK (ihrac edilmemis), bu yuzden hala tahmin.
-    Olculecek: aksa gore ileri/geri mesafe + zeminden yukseklik.
     KABUL (29.07, kullanici karari): LiDAR ust kapaga montajli ve taramasi
     engelsiz 360 derece. Boylece SLAM, AMCL ve costmap standart bir 2D
     tarayici varsayimiyla kurulabiliyor; sektor maskeleme (ignore_array)
     gerekmiyor.
-    Ust kapagin duz ust yuzeyi OLCULDU: zeminden 544.5 mm (ÜstKapak-2 ve
-    DM_Üst-1 ust yuzleri ayni duzlemde). Tmini Pro govde yuksekligi 33 mm,
-    tarama duzlemi govdenin ortasina yakin -> yuzeyin ~20 mm uzerinde.
-      lidar_z = 0.5645 - 0.100 (aks yuksekligi) = 0.4645
-    x ve y hala TAHMINI: tutucu CAD'e islenmedi. x=0.400 ust kapagin on
-    bolgesine denk geliyor (ÜstKapak-2 boylamsal olarak 0.275..0.475
-    arasini kapliyor).
+    base_link, base_footprint'in 0.100 m ustundedir. lidar_z=0.180 ile tarama
+    duzlemi base_footprint'e gore zeminden 0.280 m olur.
   -->
-  <xacro:property name="lidar_x"           value="0.400"/>
+  <xacro:property name="lidar_x"           value="-0.300"/>
   <xacro:property name="lidar_y"           value="0.000"/>
-  <xacro:property name="lidar_z"           value="0.4645"/>
+  <xacro:property name="lidar_z"           value="0.180"/>
   <!--
     On ve arka IMX219 kameralari, zemindeki seridi gormek icin asagi egimli.

File: src/marco_description/urdf/sensors.xacro (robot description, xacro)
@@ -2,5 +2,6 @@
 <robot xmlns:xacro="http://www.ros.org/wiki/xacro">
   <!--
-    Sensor cerceveleri. Buradaki konumlar TAHMINIDIR (properties.xacro).
+    Sensor cerceveleri properties.xacro'da tanimlidir. LiDAR konumu gercek
+    donanimda dogrulanmistir; kamera konumlari kendi notlarindaki durumdadir.
     laser_link ozellikle kritiktir: SLAM haritasi ve AMCL lokalizasyonu
     dogrudan bu donusum uzerinden hesaplanir. base_link'e gore birkac

Commit message: feat: complete field demo and STM32 IMU integration

File: src/marco_description/urdf/properties.xacro (robot description, xacro)
@@ -116,13 +116,12 @@
     (RPLIDAR A3 DEGIL; eldeki birim Tmini Pro, bkz. AGENT_REFERANS.md)
     laser_link dogru degilse SLAM haritasi ve AMCL lokalizasyonu kayar.
-    KABUL (29.07, kullanici karari): LiDAR ust kapaga montajli ve taramasi
-    engelsiz 360 derece. Boylece SLAM, AMCL ve costmap standart bir 2D
-    tarayici varsayimiyla kurulabiliyor; sektor maskeleme (ignore_array)
-    gerekmiyor.
-    base_link, base_footprint'in 0.100 m ustundedir. lidar_z=0.180 ile tarama
-    duzlemi base_footprint'e gore zeminden 0.280 m olur.
+    KABUL (10.08, kullanici olcumu): base_footprint'e gore LiDAR tarama
+    merkezi x=0.000, y=+0.240, z=0.280 m.
+    base_link, base_footprint'in 0.100 m ustundedir. Bu nedenle asagidaki
+    base_link'e gore z degeri 0.180 m'dir; TF zincirinde zemine gore
+    laser_link z=0.280 m olur.
   -->
-  <xacro:property name="lidar_x"           value="-0.300"/>
-  <xacro:property name="lidar_y"           value="0.000"/>
+  <xacro:property name="lidar_x"           value="0.000"/>
+  <xacro:property name="lidar_y"           value="0.240"/>
   <xacro:property name="lidar_z"           value="0.180"/>
   <!--

Commit message: stabilize mapping localization and route demo

File: src/marco_description/urdf/properties.xacro (robot description, xacro)
@@ -116,13 +116,14 @@
     (RPLIDAR A3 DEGIL; eldeki birim Tmini Pro, bkz. AGENT_REFERANS.md)
     laser_link dogru degilse SLAM haritasi ve AMCL lokalizasyonu kayar.
-    KABUL (10.08, kullanici olcumu): base_footprint'e gore LiDAR tarama
-    merkezi x=0.000, y=+0.240, z=0.280 m.
+    KABUL (11.08, kullanici fiziksel olcumu): base_footprint'e gore LiDAR
+    tarama merkezi x=+0.350, y=0.000, z=0.450 m.
     base_link, base_footprint'in 0.100 m ustundedir. Bu nedenle asagidaki
-    base_link'e gore z degeri 0.180 m'dir; TF zincirinde zemine gore
-    laser_link z=0.280 m olur.
+    base_link'e gore z degeri 0.350 m'dir; TF zincirinde zemine gore
+    laser_link z=0.450 m olur. LiDAR yaw'i olculene kadar sifir kabul edilir;
+    fiziksel montaj yonu /scan_raw ile ayrica kalibre edilmelidir.
   -->
-  <xacro:property name="lidar_x"           value="0.000"/>
-  <xacro:property name="lidar_y"           value="0.240"/>
-  <xacro:property name="lidar_z"           value="0.180"/>
+  <xacro:property name="lidar_x"           value="0.350"/>
+  <xacro:property name="lidar_y"           value="0.000"/>
+  <xacro:property name="lidar_z"           value="0.350"/>
   <!--
     On ve arka IMX219 kameralari, zemindeki seridi gormek icin asagi egimli.

File: src/marco_description/urdf/sensors.xacro (robot description, xacro)
@@ -13,4 +13,6 @@
     olarak yayinlar (marco_localization/config/lidar_tmini_pro.yaml),
     bu link ile birebir eslesir; ek static TF gerekmez.
+    rpy simdilik 0 0 0 kabuludur. Fiziksel montaj yaw'i /scan_raw ile
+    olculmeden bu donusume tahmini bir aci eklenmemelidir.
     Olculen tarama: 360 derece, 430 nokta, 0.03-12 m, 10 Hz.
     Govde olculeri yaklasiktir, gorsel amacli.

Commit message: RPLiDAR A2M12'ye geçiş

File: src/marco_description/urdf/properties.xacro (robot description, xacro)
@@ -112,18 +112,17 @@
   <!-- ==================== SENSOR YERLESIMI ==================== -->
   <!--
-    Orange Pi gercek donanim dogrulamasi: YDLidar Tmini Pro'nun base_link'e
+    Orange Pi gercek donanim dogrulamasi: RPLIDAR A2M12'nin base_link'e
     gore konumu.
-    (RPLIDAR A3 DEGIL; eldeki birim Tmini Pro, bkz. AGENT_REFERANS.md)
     laser_link dogru degilse SLAM haritasi ve AMCL lokalizasyonu kayar.
-    KABUL (11.08, kullanici fiziksel olcumu): base_footprint'e gore LiDAR
-    tarama merkezi x=+0.350, y=0.000, z=0.450 m.
+    KABUL (02.09, kullanici fiziksel olcumu): base_footprint'e gore LiDAR
+    tarama merkezi x=+0.270, y=0.000, z=0.300 m.
     base_link, base_footprint'in 0.100 m ustundedir. Bu nedenle asagidaki
-    base_link'e gore z degeri 0.350 m'dir; TF zincirinde zemine gore
-    laser_link z=0.450 m olur. LiDAR yaw'i olculene kadar sifir kabul edilir;
+    base_link'e gore z degeri 0.200 m'dir; TF zincirinde zemine gore
+    laser_link z=0.300 m olur. LiDAR yaw'i olculene kadar sifir kabul edilir;
     fiziksel montaj yonu /scan_raw ile ayrica kalibre edilmelidir.
   -->
-  <xacro:property name="lidar_x"           value="0.350"/>
+  <xacro:property name="lidar_x"           value="0.270"/>
   <xacro:property name="lidar_y"           value="0.000"/>
-  <xacro:property name="lidar_z"           value="0.350"/>
+  <xacro:property name="lidar_z"           value="0.200"/>
   <!--
     On ve arka IMX219 kameralari, zemindeki seridi gormek icin asagi egimli.

File: src/marco_description/urdf/sensors.xacro (robot description, xacro)
@@ -10,11 +10,10 @@
   -->
   <!--
-    YDLidar Tmini Pro. Surucu yapilandirmasi frame_id'yi "laser_link"
-    olarak yayinlar (marco_localization/config/lidar_tmini_pro.yaml),
-    bu link ile birebir eslesir; ek static TF gerekmez.
+    Aktif RPLIDAR A2M12 yapilandirmasi frame_id'yi "laser_link" olarak
+    yayinlar (marco_localization/config/lidar_rplidar_a2m12.yaml); bu link
+    ile birebir eslesir ve mevcut fiziksel montaj pozu korunur.
     rpy simdilik 0 0 0 kabuludur. Fiziksel montaj yaw'i /scan_raw ile
     olculmeden bu donusume tahmini bir aci eklenmemelidir.
-    Olculen tarama: 360 derece, 430 nokta, 0.03-12 m, 10 Hz.
-    Govde olculeri yaklasiktir, gorsel amacli.
+    Tarama 360 derecedir. Govde olculeri yaklasiktir, gorsel amaclidir.
   -->
   <joint name="base_link_to_laser" type="fixed">

Commit message: haritalama calısan versiyonu, eger haritalama ilerleyen versiyonlarda bozulduysa yapılan degisiklikleri kontrol edip güncel hal icin uygulayın

File: src/marco_description/urdf/properties.xacro (robot description, xacro)
@@ -120,6 +120,7 @@
     base_link, base_footprint'in 0.100 m ustundedir. Bu nedenle asagidaki
     base_link'e gore z degeri 0.200 m'dir; TF zincirinde zemine gore
-    laser_link z=0.300 m olur. LiDAR yaw'i olculene kadar sifir kabul edilir;
-    fiziksel montaj yonu /scan_raw ile ayrica kalibre edilmelidir.
+    laser_link z=0.300 m olur. Saha testinde fiziksel on, LiDAR scan
+    koordinatinda yaklasik -170..-179 derece goruldugu icin sensors.xacro
+    icindeki base_link -> laser_link yaw duzeltmesi pi'dir.
   -->
   <xacro:property name="lidar_x"           value="0.270"/>

File: src/marco_description/urdf/sensors.xacro (robot description, xacro)
@@ -13,6 +13,7 @@
     yayinlar (marco_localization/config/lidar_rplidar_a2m12.yaml); bu link
     ile birebir eslesir ve mevcut fiziksel montaj pozu korunur.
-    rpy simdilik 0 0 0 kabuludur. Fiziksel montaj yaw'i /scan_raw ile
-    olculmeden bu donusume tahmini bir aci eklenmemelidir.
+    Saha testinde arac fiziksel onundeki hedef /scan_raw icinde yaklasik
+    -170..-179 derece goruldu. Fiziksel arac onu base_link +X oldugu icin
+    base_link -> laser_link sabit donusumunde yaw=pi uygulanir.
     Tarama 360 derecedir. Govde olculeri yaklasiktir, gorsel amaclidir.
   -->
@@ -20,5 +21,5 @@
     <parent link="base_link"/>
     <child  link="laser_link"/>
-    <origin xyz="${lidar_x} ${lidar_y} ${lidar_z}" rpy="0 0 0"/>
+    <origin xyz="${lidar_x} ${lidar_y} ${lidar_z}" rpy="0 0 ${pi}"/>
   </joint>
   <link name="laser_link">

Commit message: kalibrasyon

File: src/marco_description/urdf/properties.xacro (robot description, xacro)
@@ -29,6 +29,6 @@
         z_urdf = (y_cad -   13.778) / 1000    yukari +
     Bu donusumun sonuclari:
-      tahrik tekeri x_cad=595.40 -> y=+0.230  SOL
-      tahrik tekeri x_cad=135.40 -> y=-0.230  SAG
+      tahrik tekeri merkezi -> y=+0.215  SOL
+      tahrik tekeri merkezi -> y=-0.215  SAG
       catal ucu               -> x=-1.160
       govde on yuzu           -> x=+0.477
@@ -55,9 +55,5 @@
   <xacro:property name="wheel_width"       value="0.050"/>
   <!--
-    OLCULDU: teker merkezleri x=135.40 ve x=595.40 -> 460.00 mm.
-    Onceki TAHMINI deger 0.520 idi ve %13 hataliydi. Diferansiyel odometride
-    aci hizi (v_sag - v_sol) / wheel_separation oldugu icin bu hata her donusu
-    %11.5 eksik saydiriyordu: gercek 101.7 derecelik donus 90 derece olarak
-    raporlanir. Sartnamenin +/-5 derece yon toleransi tek donuste asilirdi.
+    DOGRULANMIS: fiziksel/CAD tahrik tekeri merkez araligi 430.00 mm.
     Bu deger fiziksel model icindir. Encoder odometrisi base_driver.yaml'daki
     saha kalibrasyonlu etkin wheel_separation degerini kullanir.
@@ -66,5 +62,5 @@
     duruyor (yay serbest konumu); arac agirligi altinda basiyor.
   -->
-  <xacro:property name="wheel_separation"  value="0.460"/>
+  <xacro:property name="wheel_separation"  value="0.430"/>
   <!--
     OLCULDU: 0.475 m. base_link tahrik aksinin ortasina yerlesir (donme

Commit message: yeni araç konfigürasyonları

File: src/marco_description/urdf/properties.xacro (robot description, xacro)
@@ -43,24 +43,26 @@
   <!-- OLCULDU: zeminden en ust noktaya 544.5 mm -->
   <xacro:property name="total_height"      value="0.545"/>
-  <!-- OLCULDU: en alcak sabit nokta catal alti, zeminden 21.6 mm -->
-  <xacro:property name="ground_clearance"  value="0.022"/>
+  <!-- SAHA OLCUMU: sasi yerden 30 mm (eski CAD'de 21.6 mm). -->
+  <xacro:property name="ground_clearance"  value="0.030"/>
   <!-- OLCULDU: sasi Taban-1 ve yan paneller z 696.9..1646.9 -> 950.0 mm.
        Kalan uzunluk direk (mast, z~620) ve catallara ait. -->
   <xacro:property name="body_length"       value="0.950"/>
   <!-- ==================== TAHRIK TEKERLEKLERI ==================== -->
-  <!-- OLCULDU: kusursuz silindir, yaricap 100.00 mm, dis kabuk sacilimi
-       0.000 mm. Rapordaki 200 mm cap degeriyle birebir uyusuyor. -->
-  <xacro:property name="wheel_radius"      value="0.100"/>
+  <!-- SAHA OLCUMU: yeni tahrik tekeri capi 250 mm, yaricapi 125 mm.
+       Eski CAD ve rapor 200 mm capli tekeri gosteriyordu. -->
+  <xacro:property name="wheel_radius"      value="0.125"/>
   <!-- OLCULDU: 50.00 mm -->
   <xacro:property name="wheel_width"       value="0.050"/>
   <!--
-    DOGRULANMIS: fiziksel/CAD tahrik tekeri merkez araligi 430.00 mm.
+    GUNCEL SAHA OLCUMU: fiziksel tahrik tekeri merkez araligi 460 mm.
+    Eski CAD geometrisi 430 mm idi.
     Bu deger fiziksel model icindir. Encoder odometrisi base_driver.yaml'daki
-    saha kalibrasyonlu etkin wheel_separation degerini kullanir.
+    1080 derece saha donuslerinden turetilen gecici etkin wheel_separation
+    degerini kullanir; yaricapin duz mesafe dogrulamasi bekleniyor.
     Tahrik uniteleri yayli: 4 adet 3 mm telli, Ø20 mm sarimli, 75 mm serbest
     boy helezon yay, akssin uzerinde. CAD'de teker zeminden 11.5 mm yukarida
     duruyor (yay serbest konumu); arac agirligi altinda basiyor.
   -->
-  <xacro:property name="wheel_separation"  value="0.430"/>
+  <xacro:property name="wheel_separation"  value="0.460"/>
   <!--
     OLCULDU: 0.475 m. base_link tahrik aksinin ortasina yerlesir (donme
@@ -112,15 +114,15 @@
     gore konumu.
     laser_link dogru degilse SLAM haritasi ve AMCL lokalizasyonu kayar.
-    KABUL (02.09, kullanici fiziksel olcumu): base_footprint'e gore LiDAR
-    tarama merkezi x=+0.270, y=0.000, z=0.300 m.
-    base_link, base_footprint'in 0.100 m ustundedir. Bu nedenle asagidaki
-    base_link'e gore z degeri 0.200 m'dir; TF zincirinde zemine gore
-    laser_link z=0.300 m olur. Saha testinde fiziksel on, LiDAR scan
+    GUNCEL SAHA OLCUMU: base_footprint'e gore LiDAR tarama merkezi
+    x=+0.370, y=0.000, z=0.320 m.
+    base_link, base_footprint'in 0.125 m ustundedir. Bu nedenle asagidaki
+    base_link'e gore z degeri 0.195 m'dir; TF zincirinde zemine gore
+    laser_link z=0.320 m olur. Saha testinde fiziksel on, LiDAR scan
     koordinatinda yaklasik -170..-179 derece goruldugu icin sensors.xacro
     icindeki base_link -> laser_link yaw duzeltmesi pi'dir.
   -->
-  <xacro:property name="lidar_x"           value="0.270"/>
+  <xacro:property name="lidar_x"           value="0.370"/>
   <xacro:property name="lidar_y"           value="0.000"/>
-  <xacro:property name="lidar_z"           value="0.200"/>
+  <xacro:property name="lidar_z"           value="0.195"/>
   <!--
     On ve arka IMX219 kameralari, zemindeki seridi gormek icin asagi egimli.
@@ -128,5 +130,6 @@
     manevrasinda (geri surus) serit takibini o yapar; sartname madde 5.
     Bu degerler base_link'e GORE, yani zeminden yukseklik icin wheel_radius
-    (0.100) eklenmeli.
+    (0.125) eklenmeli. Kamera yuksekligi yeni saha geometrisinde yeniden
+    olculmedigi icin asagidaki eski CAD ofsetleri simdilik korunuyor.
     OLCULDU (on kamera): OnAltKapak-1 panelinde tek kamera acikligi var,
     60 x 54 mm, merkezi y=+0.3 mm (govde ortasi) ve zeminden 191.5 mm.
@@ -134,5 +137,5 @@
     70 x 90 mm iki acikligi kamera sanmayin, onlar sarhos tekerlerin
     onunu aciyor.
-    -> camera_front_z = 0.1915 - 0.100 = 0.0915
+    -> eski CAD: camera_front_z = 0.1915 - 0.100 = 0.0915
     Onceki tahmin 0.350 (zeminden 0.450) idi; 26 cm sapma vardi. Kameranin
     zeminde gordugu bolge yukseklikle dogrudan olceklendigi icin serit

Commit message: odometri mapping araç konfigürasyon  güncellemeleri

File: src/marco_description/urdf/properties.xacro (robot description, xacro)
@@ -49,7 +49,7 @@
   <xacro:property name="body_length"       value="0.950"/>
   <!-- ==================== TAHRIK TEKERLEKLERI ==================== -->
-  <!-- SAHA OLCUMU: yeni tahrik tekeri capi 250 mm, yaricapi 125 mm.
-       Eski CAD ve rapor 200 mm capli tekeri gosteriyordu. -->
-  <xacro:property name="wheel_radius"      value="0.125"/>
+  <!-- Nominal teker capi 250 mm; duz saha kalibrasyonundan etkin
+       yuvarlanma yaricapi 117.7 mm olarak belirlendi. -->
+  <xacro:property name="wheel_radius"      value="0.1177"/>
   <!-- OLCULDU: 50.00 mm -->
   <xacro:property name="wheel_width"       value="0.050"/>
@@ -58,6 +58,6 @@
     Eski CAD geometrisi 430 mm idi.
     Bu deger fiziksel model icindir. Encoder odometrisi base_driver.yaml'daki
-    1080 derece saha donuslerinden turetilen gecici etkin wheel_separation
-    degerini kullanir; yaricapin duz mesafe dogrulamasi bekleniyor.
+    1080 derece saha donusleri ve duz mesafe olcumunden turetilen etkin
+    wheel_separation degerini kullanir.
     Tahrik uniteleri yayli: 4 adet 3 mm telli, Ø20 mm sarimli, 75 mm serbest
     boy helezon yay, akssin uzerinde. CAD'de teker zeminden 11.5 mm yukarida
@@ -116,6 +116,6 @@
     GUNCEL SAHA OLCUMU: base_footprint'e gore LiDAR tarama merkezi
     x=+0.370, y=0.000, z=0.320 m.
-    base_link, base_footprint'in 0.125 m ustundedir. Bu nedenle asagidaki
-    base_link'e gore z degeri 0.195 m'dir; TF zincirinde zemine gore
+    base_link, base_footprint'in 0.1177 m ustundedir. Bu nedenle asagidaki
+    base_link'e gore z degeri 0.2023 m'dir; TF zincirinde zemine gore
     laser_link z=0.320 m olur. Saha testinde fiziksel on, LiDAR scan
     koordinatinda yaklasik -170..-179 derece goruldugu icin sensors.xacro
@@ -124,5 +124,5 @@
   <xacro:property name="lidar_x"           value="0.370"/>
   <xacro:property name="lidar_y"           value="0.000"/>
-  <xacro:property name="lidar_z"           value="0.195"/>
+  <xacro:property name="lidar_z"           value="0.2023"/>
   <!--
     On ve arka IMX219 kameralari, zemindeki seridi gormek icin asagi egimli.
@@ -130,5 +130,5 @@
     manevrasinda (geri surus) serit takibini o yapar; sartname madde 5.
     Bu degerler base_link'e GORE, yani zeminden yukseklik icin wheel_radius
-    (0.125) eklenmeli. Kamera yuksekligi yeni saha geometrisinde yeniden
+    (0.1177) eklenmeli. Kamera yuksekligi yeni saha geometrisinde yeniden
     olculmedigi icin asagidaki eski CAD ofsetleri simdilik korunuyor.
     OLCULDU (on kamera): OnAltKapak-1 panelinde tek kamera acikligi var,

Commit message: getgraph bugfix

File: src/marco_description/urdf/properties.xacro (robot description, xacro)
@@ -49,7 +49,6 @@
   <xacro:property name="body_length"       value="0.950"/>
   <!-- ==================== TAHRIK TEKERLEKLERI ==================== -->
-  <!-- Nominal teker capi 250 mm; duz saha kalibrasyonundan etkin
-       yuvarlanma yaricapi 117.7 mm olarak belirlendi. -->
-  <xacro:property name="wheel_radius"      value="0.1177"/>
+  <!-- Nominal teker capi 250 mm; yuvarlanma yaricapi 125 mm. -->
+  <xacro:property name="wheel_radius"      value="0.125"/>
   <!-- OLCULDU: 50.00 mm -->
   <xacro:property name="wheel_width"       value="0.050"/>
@@ -57,7 +56,6 @@
     GUNCEL SAHA OLCUMU: fiziksel tahrik tekeri merkez araligi 460 mm.
     Eski CAD geometrisi 430 mm idi.
-    Bu deger fiziksel model icindir. Encoder odometrisi base_driver.yaml'daki
-    1080 derece saha donusleri ve duz mesafe olcumunden turetilen etkin
-    wheel_separation degerini kullanir.
+    Fiziksel model ve encoder odometrisi ayni wheel_separation degerini
+    kullanir.
     Tahrik uniteleri yayli: 4 adet 3 mm telli, Ø20 mm sarimli, 75 mm serbest
     boy helezon yay, akssin uzerinde. CAD'de teker zeminden 11.5 mm yukarida
@@ -116,6 +114,6 @@
     GUNCEL SAHA OLCUMU: base_footprint'e gore LiDAR tarama merkezi
     x=+0.370, y=0.000, z=0.320 m.
-    base_link, base_footprint'in 0.1177 m ustundedir. Bu nedenle asagidaki
-    base_link'e gore z degeri 0.2023 m'dir; TF zincirinde zemine gore
+    base_link, base_footprint'in 0.125 m ustundedir. Bu nedenle asagidaki
+    base_link'e gore z degeri 0.195 m'dir; TF zincirinde zemine gore
     laser_link z=0.320 m olur. Saha testinde fiziksel on, LiDAR scan
     koordinatinda yaklasik -170..-179 derece goruldugu icin sensors.xacro
@@ -124,5 +122,5 @@
   <xacro:property name="lidar_x"           value="0.370"/>
   <xacro:property name="lidar_y"           value="0.000"/>
-  <xacro:property name="lidar_z"           value="0.2023"/>
+  <xacro:property name="lidar_z"           value="0.195"/>
   <!--
     On ve arka IMX219 kameralari, zemindeki seridi gormek icin asagi egimli.
@@ -130,5 +128,5 @@
     manevrasinda (geri surus) serit takibini o yapar; sartname madde 5.
     Bu degerler base_link'e GORE, yani zeminden yukseklik icin wheel_radius
-    (0.1177) eklenmeli. Kamera yuksekligi yeni saha geometrisinde yeniden
+    (0.125) eklenmeli. Kamera yuksekligi yeni saha geometrisinde yeniden
     olculmedigi icin asagidaki eski CAD ofsetleri simdilik korunuyor.
     OLCULDU (on kamera): OnAltKapak-1 panelinde tek kamera acikligi var,

Commit message: lidar tepede ve serit takip öncesi dönüş değişti

File: src/marco_description/urdf/properties.xacro (robot description, xacro)
@@ -113,14 +113,14 @@
     laser_link dogru degilse SLAM haritasi ve AMCL lokalizasyonu kayar.
     GUNCEL SAHA OLCUMU: base_footprint'e gore LiDAR tarama merkezi
-    x=+0.370, y=0.000, z=0.320 m.
+    x=+0.260, y=0.000, z=0.560 m.
     base_link, base_footprint'in 0.125 m ustundedir. Bu nedenle asagidaki
-    base_link'e gore z degeri 0.195 m'dir; TF zincirinde zemine gore
-    laser_link z=0.320 m olur. Saha testinde fiziksel on, LiDAR scan
+    base_link'e gore z degeri 0.435 m'dir; TF zincirinde zemine gore
+    laser_link z=0.560 m olur. Saha testinde fiziksel on, LiDAR scan
     koordinatinda yaklasik -170..-179 derece goruldugu icin sensors.xacro
     icindeki base_link -> laser_link yaw duzeltmesi pi'dir.
   -->
-  <xacro:property name="lidar_x"           value="0.370"/>
+  <xacro:property name="lidar_x"           value="0.260"/>
   <xacro:property name="lidar_y"           value="0.000"/>
-  <xacro:property name="lidar_z"           value="0.195"/>
+  <xacro:property name="lidar_z"           value="0.435"/>
   <!--
     On ve arka IMX219 kameralari, zemindeki seridi gormek icin asagi egimli.

File: src/marco_description/urdf/sensors.xacro (robot description, xacro)
@@ -12,5 +12,5 @@
     Aktif RPLIDAR A2M12 yapilandirmasi frame_id'yi "laser_link" olarak
     yayinlar (marco_localization/config/lidar_rplidar_a2m12.yaml); bu link
-    ile birebir eslesir ve mevcut fiziksel montaj pozu korunur.
+    ile birebir eslesir ve fiziksel montaj pozu URDF TF'inde temsil edilir.
     Saha testinde arac fiziksel onundeki hedef /scan_raw icinde yaklasik
     -170..-179 derece goruldu. Fiziksel arac onu base_link +X oldugu icin
