Commit message: Faz 9 docking simulasyon kabulunu tamamla

File: src/marco_simulation/urdf/marco_sim.urdf.xacro (robot description, xacro)
@@ -6,4 +6,8 @@
   <!-- Fortress clamps rays when the 3 cm minimum range overlaps the body top. -->
   <xacro:property name="lidar_z" value="0.4845"/>
+  <!-- Sim-only unobstructed camera mount; real CAD/calibration stays untouched. -->
+  <xacro:property name="camera_front_z" value="0.58"/>
+  <xacro:property name="camera_rear_z" value="0.58"/>
+  <xacro:property name="camera_pitch" value="1.10"/>
   <xacro:include filename="$(find marco_description)/urdf/common.xacro"/>
   <xacro:include filename="$(find marco_description)/urdf/base.xacro"/>
@@ -97,5 +101,8 @@
     </sensor>
   </gazebo>
-  <gazebo reference="camera_front_optical_frame">
+  <!-- Gazebo camera looks along camera_link +X. The optical frame is only the
+       ROS message frame; mounting the sensor on the already-rotated optical
+       link would apply the REP-103 rotation twice. -->
+  <gazebo reference="camera_front_link">
     <sensor name="front_camera" type="camera">
       <topic>/camera/image_raw</topic>
@@ -112,3 +119,15 @@
     </sensor>
   </gazebo>
+  <gazebo reference="camera_rear_link">
+    <sensor name="rear_camera" type="camera">
+      <topic>/camera_rear/image_raw</topic>
+      <gz_frame_id>camera_rear_optical_frame</gz_frame_id>
+      <update_rate>15</update_rate><always_on>true</always_on><visualize>true</visualize>
+      <camera><horizontal_fov>1.3962634</horizontal_fov>
+        <image><width>640</width><height>480</height><format>R8G8B8</format></image>
+        <clip><near>0.03</near><far>20.0</far></clip>
+        <camera_info_topic>/camera_rear/camera_info</camera_info_topic>
+      </camera>
+    </sensor>
+  </gazebo>
 </robot>
